File: 01_RaspberryPi-Pico-Motor-Expansion-Board_EMC_safe_design/01_RaspberryPi-Pico-Motor-Expansion-Board_EMC_safe_design.kicad_sch (KiCad schematic)
At the start: 0 parts

Commit message: update
Parts:
- added J?: USB_C_Receptacle_USB2.0_16P, symbol Connector:USB_C_Receptacle_USB2.0_16P
Connections:
- new net: J?.A1 (GND), J?.A12 (GND), J?.B1 (GND), J?.B12 (GND)
- new net: J?.A4 (VBUS), J?.A9 (VBUS), J?.B4 (VBUS), J?.B9 (VBUS)
Changed lines of the file:
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@@
 	(generator_version "9.0")
 	(paper "A4")
+	(symbol
+		(lib_id "Connector:USB_C_Receptacle_USB2.0_16P")
+		(at 73.66 69.85 0)
+		(unit 1)
+		(exclude_from_sim no)
+		(in_bom yes)
+		(on_board yes)
+		(dnp no)
+		(fields_autoplaced yes)
+		(property "Reference" "J?"
+			(at 73.66 46.99 0)
+			(effects
+				(font
+					(size 1.27 1.27)
+				)
+			)
+		)
+		(property "Value" "USB_C_Receptacle_USB2.0_16P"
+			(at 73.66 49.53 0)
+			(effects
+				(font
+					(size 1.27 1.27)
+				)
+			)
+		)
+		(property "Footprint" ""
+			(at 77.47 69.85 0)
+			(effects
+				(font
+					(size 1.27 1.27)
+				)
+				(hide yes)
+			)
+		)
+		(property "Datasheet" "https://www.usb.org/sites/default/files/documents/usb_type-c.zip"
+			(at 77.47 69.85 0)
+			(effects
+				(font
+					(size 1.27 1.27)
+				)
+				(hide yes)
+			)
+		)
+		(property "Description" "USB 2.0-only 16P Type-C Receptacle connector"
+			(at 73.66 69.85 0)
+			(effects
+				(font
+					(size 1.27 1.27)
+				)
+				(hide yes)
+			)
+		)
+		(pin "S1"
+		)
+		(pin "A1"
+		)
+		(pin "A12"
+		)
+		(pin "B1"
+		)
+		(pin "B12"
+		)
+		(pin "A4"
+		)
+		(pin "A9"
+		)
+		(pin "B4"
+		)
+		(pin "B9"
+		)
+		(pin "A5"
+		)
+		(pin "B5"
+		)
+		(pin "A7"
+		)
+		(pin "B7"
+		)
+		(pin "A6"
+		)
+		(pin "B6"
+		)
+		(pin "A8"
+		)
+		(pin "B8"
+		)
+		(instances
+			(project ""
+				(path "/4489f03b-fc05-472b-b2d8-0e342d5c95b9"
+					(reference "J?")
+					(unit 1)
+				)
+			)
+		)
+	)
 	(sheet_instances
 		(path "/"
